Commit message: [ergoCubSN000] Fix the torso pitch to 10deg

File: urdf/ergoCub/robots/ergoCubSN000/model.urdf (robot description, URDF)
Before this commit: robot ergoCub, 193 links, 192 joints
Joints:
- joint torso_pitch: origin xyz=0 0 0.11800000000000005 rpy=0 0 0 -> xyz=0 0 0.11800000000000005 rpy=0 0.174533 0
